Commit message: correct ball_chaser and urdf model

File: catkin_ws/src/my_robot/urdf/my_robot.xacro (robot description, xacro)
@@ -35,5 +35,5 @@
       <origin xyz="-0.15 0 -0.05" rpy=" 0 0 0"/>
       <geometry>
-        <sphere radius="0.0499"/>
+        <sphere radius="0.05"/>
       </geometry>
     </collision>
@@ -47,5 +47,5 @@
       <origin xyz="0.15 0 -0.05" rpy=" 0 0 0"/>
       <geometry>
-        <sphere radius="0.0499"/>
+        <sphere radius="0.05"/>
       </geometry>
     </collision>
@@ -60,5 +60,5 @@
   <link name="left_wheel">
     <collision name="left_wheel_collision">
-      <origin xyz="0 0 0" rpy="0 1.57 1.57"/>
+      <origin xyz="0 0 0" rpy="0 0 0"/>
       <geometry>
         <cylinder radius="0.1" length="0.05"/>
@@ -66,5 +66,5 @@
     </collision>
     <visual name="left_wheel_visual">
-      <origin xyz="0 0 0" rpy="0 1.57 1.57"/>
+      <origin xyz="0 0 0" rpy="0 0 0"/>
       <geometry>
         <cylinder radius="0.1" length="0.05"/>
@@ -72,5 +72,5 @@
     </visual>
     <inertial>
-      <origin xyz="0 0 0" rpy="0 1.57 1.57"/>
+      <origin xyz="0 0 0" rpy="0 0 0"/>
       <mass value="5"/>
       <inertia
@@ -84,5 +84,5 @@
   <link name="right_wheel">
     <collision name="right_wheel_collision">
-      <origin xyz="0 0 0" rpy="0 1.57 1.57"/>
+      <origin xyz="0 0 0" rpy="0 0 0"/>
       <geometry>
         <cylinder radius="0.1" length="0.05"/>
@@ -90,5 +90,5 @@
     </collision>
     <visual name="right_wheel_visual">
-      <origin xyz="0 0 0" rpy="0 1.57 1.57"/>
+      <origin xyz="0 0 0" rpy="0 0 0"/>
       <geometry>
         <cylinder radius="0.1" length="0.05"/>
@@ -96,5 +96,5 @@
     </visual>
     <inertial>
-      <origin xyz="0 0 0" rpy="0 1.57 1.57"/>
+      <origin xyz="0 0 0" rpy="0 0 0"/>
       <mass value="5"/>
       <inertia
@@ -107,8 +107,8 @@
   <!-- chassis to left wheel joint -->
   <joint type="continuous" name="left_wheel_hinge">
-    <origin xyz="0 0.15 0" rpy="0 0 0"/>
+    <origin xyz="0 0.15 0" rpy="1.57 0 0"/>
     <child link="left_wheel"/>
     <parent link="chassis"/>
-    <axis xyz="0 1 0" rpy="0 0 0"/>
+    <axis xyz="0 0 -1" rpy="0 0 0"/>
     <limit effort="10000" velocity="1000"/>
     <dynamics damping="1.0" friction="1.0"/>
@@ -116,8 +116,8 @@
   <!-- chassis to right wheel joint -->
   <joint type="continuous" name="right_wheel_hinge">
-    <origin xyz="0 -0.15 0" rpy="0 0 0"/>
+    <origin xyz="0 -0.15 0" rpy="-1.57 0 0"/>
     <child link="right_wheel"/>
     <parent link="chassis"/>
-    <axis xyz="0 -1 0" rpy="0 0 0"/>
+    <axis xyz="0 0 1" rpy="0 0 0"/>
     <limit effort="10000" velocity="1000"/>
     <dynamics damping="1.0" friction="1.0"/>

Commit message: final corrections

File: catkin_ws/src/my_robot/urdf/my_robot.xacro (robot description, xacro)
@@ -12,5 +12,5 @@
     <pose>0 0 0.1 0 0 0</pose>
     <inertial>
-      <mass value="15.0"/>
+      <mass value="10.0"/>
       <origin xyz="0.0 0 0" rpy=" 0 0 0"/>
       <inertia
@@ -23,5 +23,5 @@
       <origin xyz="0 0 0" rpy=" 0 0 0"/>
       <geometry>
-        <box size=".4 .2 .1"/>
+        <cylinder radius="0.3" length="0.05"/>
       </geometry>
     </collision>
@@ -29,5 +29,5 @@
       <origin xyz="0 0 0" rpy=" 0 0 0"/>
       <geometry>
-        <box size=".4 .2 .1"/>
+        <cylinder radius="0.3" length="0.05"/>
       </geometry>
     </visual>
@@ -107,5 +107,5 @@
   <!-- chassis to left wheel joint -->
   <joint type="continuous" name="left_wheel_hinge">
-    <origin xyz="0 0.15 0" rpy="1.57 0 0"/>
+    <origin xyz="0 0.35 0" rpy="1.57 0 0"/>
     <child link="left_wheel"/>
     <parent link="chassis"/>
@@ -116,5 +116,5 @@
   <!-- chassis to right wheel joint -->
   <joint type="continuous" name="right_wheel_hinge">
-    <origin xyz="0 -0.15 0" rpy="-1.57 0 0"/>
+    <origin xyz="0 -0.35 0" rpy="-1.57 0 0"/>
     <child link="right_wheel"/>
     <parent link="chassis"/>
@@ -148,5 +148,5 @@
   <!-- chassis to camera joint -->
   <joint type="fixed" name="camera_joint">
-    <origin xyz="0.2 0 0" rpy="0 0 0"/>
+    <origin xyz="0.4 0 0" rpy="0 0 0"/>
     <child link="camera"/>
     <parent link="chassis"/>
@@ -184,14 +184,11 @@
   </joint>
   <gazebo reference="left_wheel">
-    <material>Gazebo/Green</material>
+    <material>Gazebo/Orange</material>
   </gazebo>
   <gazebo reference="right_wheel">
-    <material>Gazebo/Green</material>
+    <material>Gazebo/Orange</material>
   </gazebo>
   <gazebo reference="chassis">
-    <material>Gazebo/Blue</material>
-  </gazebo>
-  <gazebo reference="camera">
-    <material>Gazebo/Red</material>
+    <material>Gazebo/Yellow</material>
   </gazebo>
 </robot>
